Commit message: Adding XACRO SUPORT

File: box_car_description/robot/box_bot_propeller.xacro (robot description, xacro)
@@ -18,5 +18,5 @@
           <origin rpy="0 0 0" xyz="0 0.0 0.0" />
           <geometry>
-            <mesh filename="package://box_bot_description/meshes/prop.stl" scale="1.0 1.0 1.0"/>
+            <mesh filename="package://box_car_description/meshes/prop.stl" scale="1.0 1.0 1.0"/>
           </geometry>
         </visual>
