Commit message: Added moving steering wheels version 1

File: box_car_description/robot/box_bot.xacro (robot description, xacro)
@@ -8,4 +8,6 @@
   <xacro:include filename="$(find box_car_description)/robot/box_bot_body.xacro" />
   <xacro:include filename="$(find box_car_description)/robot/box_bot.gazebo" />
+  <!-- Extra elemenst for car -->
+  <xacro:include filename="$(find box_car_description)/robot/box_bot_body_steering.xacro" />
   <!--
   <xacro:include filename="$(find box_car_description)/robot/box_bot_propeller.xacro" />
@@ -16,5 +18,67 @@
   <xacro:link_wheel name="left_wheel" r="${wheel_radius}" l="${wheel_width}" incr="${wheel_increment}"/>
   <xacro:joint_wheel name="joint_left_wheel" parent="${base_name}" child="left_wheel" origin_xyz="0 ${-1.0 * base_box_x / 2.0} ${-1.0 * wheel_radius}" />
-  <xacro:caster_wheel parent="chassis" caster_wheel_name="front" origin_xyz="${(base_box_x / 2.0) - wheel_increment} 0 ${-1.0* base_box_x / 2.0}" radius="${wheel_increment}" legth="${dummy_length}"/>
+  <!-- <xacro:caster_wheel parent="chassis" caster_wheel_name="front" origin_xyz="${(base_box_x / 2.0) - wheel_increment} 0 ${-1.0* base_box_x / 2.0}" radius="${wheel_increment}" legth="${dummy_length}"/>
   <xacro:caster_wheel parent="chassis" caster_wheel_name="back" origin_xyz="${(-1.0 *base_box_x / 2.0) + wheel_increment} 0 ${-1.0* base_box_x / 2.0}" radius="${wheel_increment}" legth="${dummy_length}"/>
+   -->
+  <xacro:box_bot_body_steering parent_name="${base_name}" name="body_steering" origin_xyz="${base_box_x} 0 0"/>
+  <link name ='wheel_stir_right'>
+    <visual>
+      <origin xyz="0 0 0" rpy="0 0 0"/>
+      <geometry>
+        <box size="${steering_joint_length} ${steering_joint_length} ${steering_joint_length}"/>
+      </geometry>
+    </visual>
+      <inertial>
+          <origin xyz="0 0 0" rpy="0 0 0"/>
+          <mass value="0.001" />
+          <inertia ixx="4.166666666666667e-08" ixy="0.0" ixz="0.0" iyy="4.166666666666667e-08" iyz="0.0" izz="4.166666666666667e-08"/>
+      </inertial>
+  </link>
+  <xacro:steering_joint name1='body_steering' name2='wheel_stir_right' posxyz='0 ${1.0 * base_box_x / 2.0} ${-1.0 * wheel_radius}' posrpy='0 0 0' rot='0 0 1' limlow='-0.6108' limhigh='0.6108' limef='1500.0' limvel='2.0' fr='100.0' dm='100.0' />
+  <xacro:link_wheel name="front_right_wheel" r="${wheel_radius}" l="${wheel_width}" incr="${wheel_increment}"/>
+  <xacro:joint_wheel name="joint_front_right_wheel" parent="wheel_stir_right" child="front_right_wheel" origin_xyz="0 ${steering_joint_length} 0" />
+  <link name ='wheel_stir_left'>
+    <visual>
+      <origin xyz="0 0 0" rpy="0 0 0"/>
+      <geometry>
+        <box size="${steering_joint_length} ${steering_joint_length} ${steering_joint_length}"/>
+      </geometry>
+    </visual>
+      <inertial>
+          <origin xyz="0 0 0" rpy="0 0 0"/>
+          <mass value="0.001" />
+          <inertia ixx="4.166666666666667e-08" ixy="0.0" ixz="0.0" iyy="4.166666666666667e-08" iyz="0.0" izz="4.166666666666667e-08"/>
+      </inertial>
+  </link>
+  <xacro:steering_joint name1='body_steering' name2='wheel_stir_left' posxyz='0 ${-1.0 * base_box_x / 2.0} ${-1.0 * wheel_radius}' posrpy='0 0 0' rot='0 0 1' limlow='-0.6108' limhigh='0.6108' limef='1500.0' limvel='2.0' fr='100.0' dm='100.0' />
+  <xacro:link_wheel name="front_left_wheel" r="${wheel_radius}" l="${wheel_width}" incr="${wheel_increment}"/>
+  <xacro:joint_wheel name="joint_front_left_wheel" parent="wheel_stir_left" child="front_left_wheel" origin_xyz="0 ${-1.0 * steering_joint_length} 0" />
+  <ros2_control name="GazeboSystem" type="system">
+    <hardware>
+      <plugin>gazebo_ros2_control/GazeboSystem</plugin>
+    </hardware>
+    <joint name="body_steering__wheel_stir_right">
+      <command_interface name="velocity">
+        <param name="min">-10</param>
+        <param name="max">10</param>
+      </command_interface>
+      <state_interface name="position"/>
+      <state_interface name="velocity"/>
+      <state_interface name="effort"/>
+    </joint>
+    <joint name="body_steering__wheel_stir_left">
+      <command_interface name="velocity">
+        <param name="min">-10</param>
+        <param name="max">10</param>
+      </command_interface>
+      <state_interface name="position"/>
+      <state_interface name="velocity"/>
+      <state_interface name="effort"/>
+    </joint>
+  </ros2_control>
+  <gazebo>
+    <plugin filename="libgazebo_ros2_control.so" name="gazebo_ros2_control">
+      <parameters>$(find box_car_description)/config/steering_controller_velocity.yaml</parameters>
+    </plugin>
+  </gazebo>
 </robot>

File: box_car_description/robot/properties.xacro (robot description, xacro)
@@ -19,3 +19,5 @@
     <!--Caster Wheels-->
     <xacro:property name="dummy_length" value="0.001"/>
+    <!--Steering Joints Links-->
+    <xacro:property name="steering_joint_length" value="0.005"/>
 </robot>

File: box_car_description/robot/wheels.xacro (robot description, xacro)
@@ -33,3 +33,15 @@
     </joint>
   </xacro:macro >
+  <!-- EXtra steering classes -->
+  <xacro:macro name="steering_joint" params="name1 name2 posxyz posrpy rot limlow limhigh limef limvel fr dm">
+      <joint name="${name1}__${name2}" type="revolute">
+        <parent link="${name1}"/>
+        <child link="${name2}"/>
+          <origin xyz="${posxyz}" rpy="${posrpy}"/>
+          <limit lower="${limlow}" upper="${limhigh}" effort="${limef}" velocity="${limvel}"/>
+          <axis xyz="${rot}"/>
+          <!-- TODO: When setting thes evalues, joint breaks -->
+          <!-- <dynamics friction="${fr}" damping="${dm}"/> -->
+    </joint>
+  </xacro:macro>
 </robot>

Commit message: Created Steering with script and added meshes custom

File: box_car_description/robot/box_bot.xacro (robot description, xacro)
@@ -35,5 +35,5 @@
       </inertial>
   </link>
-  <xacro:steering_joint name1='body_steering' name2='wheel_stir_right' posxyz='0 ${1.0 * base_box_x / 2.0} ${-1.0 * wheel_radius}' posrpy='0 0 0' rot='0 0 1' limlow='-0.6108' limhigh='0.6108' limef='1500.0' limvel='2.0' fr='100.0' dm='100.0' />
+  <xacro:steering_joint name1='body_steering' name2='wheel_stir_right' posxyz='0 ${1.0 * base_box_x / 2.0} ${-1.0 * wheel_radius}' posrpy='0 0 0' rot='0 0 1' limlow='-0.6108' limhigh='0.6108' limef='${steer_force}' limvel='${steer_vel}' fr='${steer_fric}' dm='${steer_amort}' />
   <xacro:link_wheel name="front_right_wheel" r="${wheel_radius}" l="${wheel_width}" incr="${wheel_increment}"/>
   <xacro:joint_wheel name="joint_front_right_wheel" parent="wheel_stir_right" child="front_right_wheel" origin_xyz="0 ${steering_joint_length} 0" />
@@ -51,8 +51,9 @@
       </inertial>
   </link>
-  <xacro:steering_joint name1='body_steering' name2='wheel_stir_left' posxyz='0 ${-1.0 * base_box_x / 2.0} ${-1.0 * wheel_radius}' posrpy='0 0 0' rot='0 0 1' limlow='-0.6108' limhigh='0.6108' limef='1500.0' limvel='2.0' fr='100.0' dm='100.0' />
+  <xacro:steering_joint name1='body_steering' name2='wheel_stir_left' posxyz='0 ${-1.0 * base_box_x / 2.0} ${-1.0 * wheel_radius}' posrpy='0 0 0' rot='0 0 1' limlow='${steer_limlow}' limhigh='${steer_limhigh}' limef='${steer_force}' limvel='${steer_vel}' fr='${steer_fric}' dm='${steer_amort}' />
   <xacro:link_wheel name="front_left_wheel" r="${wheel_radius}" l="${wheel_width}" incr="${wheel_increment}"/>
   <xacro:joint_wheel name="joint_front_left_wheel" parent="wheel_stir_left" child="front_left_wheel" origin_xyz="0 ${-1.0 * steering_joint_length} 0" />
-  <ros2_control name="GazeboSystem" type="system">
+  <!-- Velocity Config -->
+  <!-- <ros2_control name="GazeboSystem" type="system">
     <hardware>
       <plugin>gazebo_ros2_control/GazeboSystem</plugin>
@@ -76,8 +77,33 @@
       <state_interface name="effort"/>
     </joint>
+  </ros2_control> -->
+  <!-- Position Config -->
+    <ros2_control name="GazeboSystem" type="system">
+    <hardware>
+      <plugin>gazebo_ros2_control/GazeboSystem</plugin>
+    </hardware>
+    <joint name="body_steering__wheel_stir_right">
+      <command_interface name="position">
+        <param name="min">${steer_limlow}</param>
+        <param name="max">${steer_limhigh}</param>
+      </command_interface>
+      <state_interface name="position"/>
+      <state_interface name="velocity"/>
+      <state_interface name="effort"/>
+    </joint>
+    <joint name="body_steering__wheel_stir_left">
+      <command_interface name="position">
+        <param name="min">${steer_limlow}</param>
+        <param name="max">${steer_limhigh}</param>
+      </command_interface>
+      <state_interface name="position"/>
+      <state_interface name="velocity"/>
+      <state_interface name="effort"/>
+    </joint>
   </ros2_control>
   <gazebo>
     <plugin filename="libgazebo_ros2_control.so" name="gazebo_ros2_control">
-      <parameters>$(find box_car_description)/config/steering_controller_velocity.yaml</parameters>
+      <!-- <parameters>$(find box_car_description)/config/steering_controller_velocity.yaml</parameters> -->
+      <parameters>$(find box_car_description)/config/steering_controller_position.yaml</parameters>
     </plugin>
   </gazebo>

File: box_car_description/robot/box_bot_body.xacro (robot description, xacro)
@@ -20,6 +20,9 @@
         </collision>
         <visual name="visual_${parent_name}">
+          <!-- <geometry>
+            <box size="${base_box_x} ${base_box_y} ${base_box_z}"/>
+          </geometry> -->
           <geometry>
-            <box size="${base_box_x} ${base_box_y} ${base_box_z}"/>
+            <mesh filename="/home/tgrip/TheConstruct/ros_2_playground/box_car_ws/src/box_car/box_car_description/meshes/box_car.dae" scale="1.0 1.0 1.0"/>
           </geometry>
         </visual>

File: box_car_description/robot/box_bot_body_steering.xacro (robot description, xacro)
@@ -17,9 +17,9 @@
           </geometry>
         </collision>
-        <visual name="visual_${name}">
+        <!-- <visual name="visual_${name}">
           <geometry>
             <box size="${base_box_x} ${base_box_y} ${base_box_z}"/>
           </geometry>
-        </visual>
+        </visual> -->
       </link>
       <gazebo reference="${name}">

File: box_car_description/robot/properties.xacro (robot description, xacro)
@@ -21,3 +21,9 @@
     <!--Steering Joints Links-->
     <xacro:property name="steering_joint_length" value="0.005"/>
+    <xacro:property name="steer_limlow" value="-0.6108"/>
+    <xacro:property name="steer_limhigh" value="0.6108"/>
+    <xacro:property name="steer_force" value="1000"/>
+    <xacro:property name="steer_vel" value="1.0"/>
+    <xacro:property name="steer_fric" value="2.0"/>
+    <xacro:property name="steer_amort" value="0.0"/>
 </robot>

File: box_car_description/robot/wheels.xacro (robot description, xacro)
@@ -17,6 +17,9 @@
           <visual name="link_right_wheel_visual">
             <origin rpy="0 1.5707 1.5707" xyz="0 0 0"/>
+            <!-- <geometry>
+              <cylinder length="${l}" radius="${r + incr}"/>
+            </geometry> -->
             <geometry>
-              <cylinder length="${l}" radius="${r + incr}"/>
+              <mesh filename="/home/tgrip/TheConstruct/ros_2_playground/box_car_ws/src/box_car/box_car_description/meshes/wheel.dae" scale="1.0 1.0 1.0"/>
             </geometry>
           </visual>
@@ -41,4 +44,5 @@
           <limit lower="${limlow}" upper="${limhigh}" effort="${limef}" velocity="${limvel}"/>
           <axis xyz="${rot}"/>
+          <dynamics damping="${dm}" friction="${fr}"/>
           <!-- TODO: When setting thes evalues, joint breaks -->
           <!-- <dynamics friction="${fr}" damping="${dm}"/> -->
